Commit message: add dummy camera in urdf and delete the effort parameter in urdf for simulation purpose

File: z1_description/urdf/z1.urdf.xacro (robot description, xacro)
@@ -302,7 +302,70 @@
             <self_collide>true</self_collide>
         </gazebo>
+        <!-- Depth Camera Link -->
+        <joint name="camera_joint" type="fixed">
+            <origin rpy="0 0 0" xyz="0.02 0.0 0.08" />
+            <parent link="gripperStator" />
+            <child link="camera_link" />
+        </joint>
+        <link name="camera_link">
+            <visual>
+                <origin rpy="0 0 0" xyz="0 0 0" />
+                <geometry>
+                    <box size="0.015 0.03 0.01" />
+                </geometry>
+                <material name="Grey" />
+            </visual>
+            <collision>
+                <origin rpy="0 0 0" xyz="0 0 0" />
+                <geometry>
+                    <box size="0.015 0.03 0.01" />
+                </geometry>
+            </collision>
+            <inertial>
+                <mass value="0.01" />
+                <origin rpy="0 0 0" xyz="0 0 0" />
+                <inertia
+                    ixx="0.00001" ixy="0.0" ixz="0.0"
+                    iyy="0.00001" iyz="0.0"
+                    izz="0.00001" />
+            </inertial>
+        </link>
+        <!-- Camera Optical Frame -->
+        <joint name="camera_optical_joint" type="fixed">
+            <origin rpy="-1.57079632679 0 -1.57079632679" xyz="0 0 0" />
+            <parent link="camera_link" />
+            <child link="camera_depth_optical_frame" />
+        </joint>
+        <link name="camera_depth_optical_frame" />
+        <!-- Ignition Gazebo RGBD Camera Sensor -->
+        <gazebo reference="camera_link">
+            <sensor name="rgbd_camera" type="rgbd_camera">
+                <camera>
+                    <horizontal_fov>1.5708</horizontal_fov>
+                    <image>
+                        <width>640</width>
+                        <height>480</height>
+                    </image>
+                    <clip>
+                        <near>0.05</near>
+                        <far>3.0</far>
+                    </clip>
+                </camera>
+                <always_on>1</always_on>
+                <update_rate>30</update_rate>
+                <visualize>true</visualize>
+                <topic>rgbd_camera</topic>
+                <enable_metrics>false</enable_metrics>
+            </sensor>
+        </gazebo>
     </xacro:if>
     <xacro:if value="$(arg sim_ignition)">
         <gazebo reference="world" />
+        <!-- Ignition Gazebo Sensors System Plugin -->
+        <gazebo>
+            <plugin filename="ignition-gazebo-sensors-system" name="ignition::gazebo::systems::Sensors">
+                <render_engine>ogre2</render_engine>
+            </plugin>
+        </gazebo>
         <gazebo>
             <plugin filename="libign_ros2_control-system.so"

Commit message: fix: add camera in urdf

File: z1_description/urdf/z1.urdf.xacro (robot description, xacro)
@@ -233,142 +233,111 @@
         </inertial>
     </link>
-    <xacro:if value="$(arg with_gripper)">
-        <joint name="gripperStatorLink" type="fixed">
-            <origin rpy="0 0 0" xyz="0.051 0.0 0.0" />
-            <parent link="link06" />
-            <child link="gripperStator" />
-        </joint>
-        <link name="gripperStator">
-            <visual>
-                <geometry>
-                    <mesh filename="package://z1_description/meshes/visual/z1_GripperStator.dae"
-                        scale="1 1 1" />
-                </geometry>
-                <material name="Grey" />
-            </visual>
-            <collision>
-                <geometry>
-                    <mesh filename="package://z1_description/meshes/collision/z1_GripperStator.STL"
-                        scale="1 1 1" />
-                </geometry>
-            </collision>
-            <inertial>
-                <origin rpy="0 0 0"
-                    xyz="${GripperStator_ComX} ${GripperStator_ComY} ${GripperStator_ComZ}" />
-                <mass value="${GripperStator_Mass}" />
-                <inertia
-                    ixx="${GripperStator_Ixx}" ixy="${GripperStator_Ixy}" ixz="${GripperStator_Ixz}"
-                    iyy="${GripperStator_Iyy}" iyz="${GripperStator_Iyz}"
-                    izz="${GripperStator_Izz}" />
-            </inertial>
-        </link>
-        <joint name="jointGripper" type="revolute">
-            <origin rpy="0 0 0" xyz="0.049 0.0 0" />
-            <parent link="gripperStator" />
-            <child link="gripperMover" />
-            <axis xyz="0 1 0" />
-            <dynamics damping="${jointDamping}" friction="${jointFriction}" />
-            <limit effort="${torqueMax}" velocity="${velocityMax}" lower="${Gripper_PositionMin}"
-                upper="${Gripper_PositionMax}" />
-        </joint>
-        <link name="gripperMover">
-            <visual>
-                <geometry>
-                    <mesh filename="package://z1_description/meshes/visual/z1_GripperMover.dae"
-                        scale="1 1 1" />
-                </geometry>
-                <material name="Grey" />
-            </visual>
-            <collision>
-                <geometry>
-                    <mesh filename="package://z1_description/meshes/collision/z1_GripperMover.STL"
-                        scale="1 1 1" />
-                </geometry>
-            </collision>
-            <inertial>
-                <origin rpy="0 0 0"
-                    xyz="${GripperMover_ComX} ${GripperMover_ComY} ${GripperMover_ComZ}" />
-                <mass value="${GripperMover_Mass}" />
-                <inertia
-                    ixx="${GripperMover_Ixx}" ixy="${GripperMover_Ixy}" ixz="${GripperMover_Ixz}"
-                    iyy="${GripperMover_Iyy}" iyz="${GripperMover_Iyz}"
-                    izz="${GripperMover_Izz}" />
-            </inertial>
-        </link>
-        <gazebo reference="gripperStator">
-            <self_collide>true</self_collide>
+    <!-- End Effector Disc (5mm thick, 60mm diameter) -->
+    <joint name="end_effector_disc_joint" type="fixed">
+        <origin rpy="0 1.57079632679 0" xyz="0.0535 0.0 0.0" />
+        <parent link="link06" />
+        <child link="end_effector_disc" />
+    </joint>
+    <link name="end_effector_disc">
+        <visual>
+            <origin rpy="0 0 0" xyz="0 0 0" />
+            <geometry>
+                <cylinder radius="0.03" length="0.005" />
+            </geometry>
+            <material name="Grey" />
+        </visual>
+        <collision>
+            <origin rpy="0 0 0" xyz="0 0 0" />
+            <geometry>
+                <cylinder radius="0.03" length="0.005" />
+            </geometry>
+        </collision>
+        <inertial>
+            <mass value="0.05" />
+            <origin rpy="0 0 0" xyz="0 0 0" />
+            <inertia
+                ixx="0.000008" ixy="0.0" ixz="0.0"
+                iyy="0.000008" iyz="0.0"
+                izz="0.000016" />
+        </inertial>
+    </link>
+    <!-- Depth Camera Link -->
+    <joint name="camera_joint" type="fixed">
+        <origin rpy="0 -1.57079632679 0" xyz="0 0 0.0275" />
+        <parent link="end_effector_disc" />
+        <child link="camera_link" />
+    </joint>
+    <link name="camera_link">
+        <visual>
+            <origin rpy="1.57079632679 0 1.57079632679" xyz="0 0 0" />
+            <geometry>
+                <mesh filename="package://z1_description/meshes/d435.dae" />
+            </geometry>
+            <material name="Grey" />
+        </visual>
+        <collision>
+            <origin rpy="0 0 0" xyz="0 0 0" />
+            <geometry>
+                <box size="0.015 0.03 0.01" />
+            </geometry>
+        </collision>
+        <inertial>
+            <mass value="0.564" />
+            <origin rpy="0 0 0" xyz="0 0 0" />
+            <inertia
+                ixx="0.003881243" ixy="0.0" ixz="0.0"
+                iyy="0.000498940" iyz="0.0"
+                izz="0.003879257" />
+        </inertial>
+    </link>
+    <!-- Camera Optical Frame -->
+    <joint name="camera_optical_joint" type="fixed">
+        <origin rpy="-1.57079632679 0 -1.57079632679" xyz="0 0 0" />
+        <parent link="camera_link" />
+        <child link="camera_depth_optical_frame" />
+    </joint>
+    <link name="camera_depth_optical_frame" />
+    <!-- Ignition Gazebo RGBD Camera Sensor -->
+    <gazebo reference="camera_link">
+        <sensor name="rgbd_camera" type="rgbd_camera">
+            <ignition_frame_id>camera_link</ignition_frame_id>
+            <optical_frame_id>camera_depth_optical_frame</optical_frame_id>
+            <camera>
+                <horizontal_fov>1.5708</horizontal_fov>
+                <image>
+                    <width>640</width>
+                    <height>480</height>
+                    <format>R8G8B8</format>
+                </image>
+                <clip>
+                    <near>0.01</near>
+                    <far>10.0</far>
+                </clip>
+            </camera>
+            <depth_camera>
+                <clip>
+                    <near>0.01</near>
+                    <far>10.0</far>
+                </clip>
+            </depth_camera>
+            <always_on>1</always_on>
+            <update_rate>30</update_rate>
+            <visualize>true</visualize>
+            <topic>rgbd_camera</topic>
+            <enable_metrics>false</enable_metrics>
+        </sensor>
+    </gazebo>
+    <xacro:if value="$(arg sim_ignition)">
+        <gazebo reference="world">
+            <!-- Set initial camera view to left-front view -->
+            <!-- Camera pose: x y z roll pitch yaw -->
+            <!-- Position: 1.5m forward (x), -1.5m left (y), 1.0m up (z) -->
+            <!-- Orientation: 0 roll, 0.3 pitch (slight downward), -2.356 yaw (135 deg, left-front) -->
+            <scene>
+                <ambient>0.4 0.4 0.4 1</ambient>
+                <background>0.8 0.8 0.8 1</background>
+                <shadows>true</shadows>
+            </scene>
         </gazebo>
-        <gazebo reference="gripperMover">
-            <self_collide>true</self_collide>
-        </gazebo>
-        <!-- Depth Camera Link -->
-        <joint name="camera_joint" type="fixed">
-            <origin rpy="0 0 0" xyz="0.02 0.0 0.08" />
-            <parent link="gripperStator" />
-            <child link="camera_link" />
-        </joint>
-        <link name="camera_link">
-            <visual>
-                <origin rpy="0 0 0" xyz="0 0 0" />
-                <geometry>
-                    <box size="0.015 0.03 0.01" />
-                </geometry>
-                <material name="Grey" />
-            </visual>
-            <collision>
-                <origin rpy="0 0 0" xyz="0 0 0" />
-                <geometry>
-                    <box size="0.015 0.03 0.01" />
-                </geometry>
-            </collision>
-            <inertial>
-                <mass value="0.01" />
-                <origin rpy="0 0 0" xyz="0 0 0" />
-                <inertia
-                    ixx="0.00001" ixy="0.0" ixz="0.0"
-                    iyy="0.00001" iyz="0.0"
-                    izz="0.00001" />
-            </inertial>
-        </link>
-        <!-- Camera Optical Frame -->
-        <joint name="camera_optical_joint" type="fixed">
-            <origin rpy="-1.57079632679 0 -1.57079632679" xyz="0 0 0" />
-            <parent link="camera_link" />
-            <child link="camera_depth_optical_frame" />
-        </joint>
-        <link name="camera_depth_optical_frame" />
-        <!-- Ignition Gazebo RGBD Camera Sensor -->
-        <gazebo reference="camera_link">
-            <sensor name="rgbd_camera" type="rgbd_camera">
-                <ignition_frame_id>camera_link</ignition_frame_id>
-                <optical_frame_id>camera_depth_optical_frame</optical_frame_id>
-                <camera>
-                    <horizontal_fov>1.5708</horizontal_fov>
-                    <image>
-                        <width>640</width>
-                        <height>480</height>
-                        <format>R8G8B8</format>
-                    </image>
-                    <clip>
-                        <near>0.01</near>
-                        <far>10.0</far>
-                    </clip>
-                </camera>
-                <depth_camera>
-                    <clip>
-                        <near>0.01</near>
-                        <far>10.0</far>
-                    </clip>
-                </depth_camera>
-                <always_on>1</always_on>
-                <update_rate>30</update_rate>
-                <visualize>true</visualize>
-                <topic>rgbd_camera</topic>
-                <enable_metrics>false</enable_metrics>
-            </sensor>
-        </gazebo>
-    </xacro:if>
-    <xacro:if value="$(arg sim_ignition)">
-        <gazebo reference="world" />
         <!-- Ignition Gazebo Sensors System Plugin -->
         <gazebo>
